File: hardware/board/nano-bat/coulomb-counter.sch (KiCad schematic (older format))
At the start: 10 parts, among them U401 LTC2942

Commit message: Adding 0.1.0 of board spin
Parts:
- removed JP401: Jumper_3_Bridged12, Connector_PinHeader_2.54mm:PinHeader_1x03_P2.54mm_Vertical_SMD_Pin1Left, symbol Jumper:Jumper_3_Bridged12
- added Q401, Q402, Q403: Si7615ADN, Package_SO:Vishay_PowerPAK_1212-8_Single, symbol nano-bat:Si7615ADN
- added R407, R408, R409: 10k, Resistor_SMD:R_0603_1608Metric, symbol Device:R_US
- added TP401, TP402, TP403, TP404: TestPoint, TestPoint:TestPoint_Pad_2.0x2.0mm, symbol Connector:TestPoint
- R404: footprint Resistor_SMD:R_0603_1608Metric -> Resistor_SMD:R_1206_3216Metric; Part 273-KDV06DR100ETCT-ND -> CSR1206FKR100CT-ND
Connections:
- net Vbatt_out: now also TP403.1, TP404.1
- net Vbatt_source: now also Q401.1 (S), Q401.2 (S), Q401.3 (S), Q402.1 (S), Q402.2 (S), Q402.3 (S), Q403.1 (S), Q403.2 (S), Q403.3 (S), R407.1, R408.1, R409.1, TP401.1, TP402.1; no longer R406.2
- net at R405.2: now also Q402.5 (D)
- net at R404.2: now also Q401.5 (D)
- new net: Q403.5 (D), R406.2
- new net ~SEL_500mA: Q401.4 (G), R407.2
- new net ~SEL_50mA: Q402.4 (G), R408.2
- new net ~SEL_5mA: Q403.4 (G), R409.2
Other:
- note added: "Maximum Current Ranges:\n* 10 Ohms - 5mA\n* 1 Ohm - 50mA\n* 100mOhm - 500mA"
- note removed: "Maximum Current Ranges:\n* 10 Ohms - 500mA\n* 1 Ohm - 50mA\n* 100 mOhm - 5mA"
- note removed: "The sensitivity of the system may be selected by JP401."
- moved on the sheet: C401, C402, R401, R402, R403, R404, R405, R406, U401
