File: hardware/board/nano-bat/nano-bat.kicad_pcb (KiCad board)
At the start: 2 copper layers, 160 x 106.7 mm, 97 parts, among them J101 Barrel_Jack_Switch, J102 USB_B_Mini, J103 Screw_Terminal_01x02, J104 Conn_01x02, J201 Conn_2Rows-45Pins, J301 Conn_ARM_JTAG_SWD_10, J302 Conn_01x10, J303 Conn_01x10, Q101 Q_PMOS_GSD, Q501 Q_PMOS_GSD, Q502 Q_NMOS_GSD, Q503 Q_NMOS_GSD, SW301 SW_Push, SW302 SW_Push, SW303 SW_Push, SW304 SW_Push, U201 AP3032, U301 M95256-WMN6P, U302 STM32L452CEUx, U401 LTC2942, U501 MIC2104YML-TR, U502 MCP1702

Commit message: Adding 0.1.0 of board spin
Parts:
- removed C508, C509: 0.1u, Capacitor_SMD:C_0603_1608Metric
- removed D101: D, Diode_SMD:D_SMA
- removed D301: BLU, LED_SMD:LED_0805_2012Metric
- removed D501: D_Schottky_ALT, Diode_SMD:D_SOD-323
- removed FB101, FB102: Ferrite_Bead_Small, Resistor_SMD:R_0603_1608Metric
- removed JP401: Jumper_3_Bridged12, Connector_PinHeader_2.54mm:PinHeader_1x03_P2.54mm_Vertical_SMD_Pin1Left
- removed NT501: Net-Tie_2, NetTie:NetTie-2_SMD_Pad2.0mm
- removed Q501: Q_PMOS_GSD, Package_TO_SOT_SMD:SOT-23
- removed Q502, Q503: Q_NMOS_GSD, Package_TO_SOT_SMD:SOT-23
- removed R309: 1k, Resistor_SMD:R_0603_1608Metric
- removed R505: 95.3k, Resistor_SMD:R_0603_1608Metric
- removed R506: 15k, Resistor_SMD:R_0603_1608Metric
- removed R507: 3.9k, Resistor_SMD:R_0603_1608Metric
- removed R508: 10.5k, Resistor_SMD:R_0603_1608Metric
- added C101: 10n, Capacitor_SMD:C_0603_1608Metric, B.Cu at (186.2, 53.6)
- added C102: 0.1u, Capacitor_SMD:C_0603_1608Metric, B.Cu at (176.0, 61.6)
- added F501: Polyfuse, Fuse:Fuse_1812_4532Metric, B.Cu at (185.2, 98.0)
- added G***: LOGO, footprints:vertigo-designs-logo, F.Cu at (188.5, 109.9)
- added H101: e, MountingHole:MountingHole_2.2mm_M2_Pad, F.Cu at (125.7, 54.6)
- added H102: e, MountingHole:MountingHole_2.2mm_M2_Pad, F.Cu at (125.7, 111.8)
- added H103: e, MountingHole:MountingHole_2.2mm_M2_Pad, F.Cu at (198.8, 111.8)
- added H104: e, MountingHole:MountingHole_2.2mm_M2_Pad, F.Cu at (198.8, 54.6)
- added Q102: Q_PMOS_GSD, Package_TO_SOT_SMD:SOT-23, F.Cu at (174.3, 68.1)
- added Q401: Si7615ADN, Package_SO:Vishay_PowerPAK_1212-8_Single, B.Cu at (181.4, 87.1)
- added Q402: Si7615ADN, Package_SO:Vishay_PowerPAK_1212-8_Single, B.Cu at (185.4, 87.1)
- added Q403: Si7615ADN, Package_SO:Vishay_PowerPAK_1212-8_Single, B.Cu at (190.9, 92.3)
- added R104: 5.1k, Resistor_SMD:R_0603_1608Metric, B.Cu at (182.9, 62.5)
- added R105: 5.1k, Resistor_SMD:R_0603_1608Metric, B.Cu at (178.6, 54.7)
- added R315: 40.2k, Resistor_SMD:R_0603_1608Metric, B.Cu at (135.8, 71.4)
- added R316: 10k, Resistor_SMD:R_0603_1608Metric, B.Cu at (136.8, 68.4)
- added R407: 10k, Resistor_SMD:R_0603_1608Metric, B.Cu at (180.3, 91.2)
- added R408: 10k, Resistor_SMD:R_0603_1608Metric, B.Cu at (184.4, 91.1)
- added R409: 10k, Resistor_SMD:R_0603_1608Metric, B.Cu at (187.9, 91.1)
- added REF**: Symbol_Barrel_Polarity, Symbol:Symbol_Barrel_Polarity, F.Cu at (190.8, 54.9)
- added REF**: OSHW-Logo2_7.3x6mm_SilkScreen, Symbol:OSHW-Logo2_7.3x6mm_SilkScreen, B.Cu at (191.9, 110.7)
- added TP301: TestPoint, TestPoint:TestPoint_THTPad_D1.0mm_Drill0.5mm, F.Cu at (134.7, 74.4)
- added TP302: TestPoint, TestPoint:TestPoint_Pad_D1.0mm, B.Cu at (148.1, 72.6)
- added TP303: TestPoint, TestPoint:TestPoint_Pad_D1.0mm, B.Cu at (145.7, 73.9)
- added TP304: TestPoint, TestPoint:TestPoint_Pad_D1.0mm, B.Cu at (162.9, 72.8)
- added TP305: TestPoint, TestPoint:TestPoint_Pad_D1.0mm, B.Cu at (167.3, 78.2)
- added TP306: TestPoint, TestPoint:TestPoint_Pad_D1.0mm, B.Cu at (154.4, 62.4)
- added TP401: TestPoint, TestPoint:TestPoint_Pad_2.0x2.0mm, B.Cu at (181.1, 94.9)
- added TP402: TestPoint, TestPoint:TestPoint_Pad_2.0x2.0mm, B.Cu at (177.0, 85.3)
- added TP403: TestPoint, TestPoint:TestPoint_Pad_2.0x2.0mm, B.Cu at (181.1, 69.6)
- added TP404: TestPoint, TestPoint:TestPoint_Pad_2.0x2.0mm, B.Cu at (177.0, 74.7)
- added U101: USBLC6-2SC6, Package_TO_SOT_SMD:SOT-23-6, B.Cu at (178.9, 61.5)
- C201, C202, C301, C302, C303, C304, C305, C306, C307, C308, C309, C310, C311, C312, C401, C402, C504, C505, C506, D201, F102, FB103, FB301, FB302, J301, L201, R201, R301, R302, R303, R304, R305, R306, R307, R308, R310, R312, R313, R314, R401, R402, R403, R405, R406, R501, U201, U301, U302, U401, U502: moved to B.Cu
- C501, C507: value 0.1u -> 10u; footprint Capacitor_SMD:C_0603_1608Metric -> Capacitor_SMD:C_0805_2012Metric; moved to B.Cu
- C502: value 4.7u -> 0.1u; moved to B.Cu
- C503: value 1u -> 0.1u; moved to B.Cu
- C510: value 4.7u -> 10u; footprint Capacitor_SMD:C_0603_1608Metric -> Capacitor_SMD:C_0805_2012Metric; moved to B.Cu
- J102: value USB_B_Mini -> USB_C_Receptacle_USB2.0; footprint footprints:USB-MICRO-B-HIROSE-UX60-MB-5S8 -> Connector_USB:USB_C_Receptacle_GCT_USB4085
- L501: value 50u -> 4.7u; footprint footprints:NRS6028-IND-NS -> Inductor_SMD:L_Taiyo-Yuden_NR-60xx; moved to B.Cu
- R101: value 1k -> 1M; moved to B.Cu
- R102: value 100k -> 1M; moved to B.Cu
- R404: footprint Resistor_SMD:R_0603_1608Metric -> Resistor_SMD:R_1206_3216Metric; moved to B.Cu
- R502: value 10k -> 1.96k; moved to B.Cu
- R503: value 10k -> 9.31k; moved to B.Cu
- R504: value 2.2k -> 10k; moved to B.Cu
- U501: value MIC2104YML-TR -> TPS562201; footprint Package_DFN_QFN:QFN-16-1EP_3x3mm_P0.5mm_EP1.7x1.7mm -> Package_TO_SOT_SMD:SOT-23-6; moved to B.Cu
- moved U302 174.8 mm to (144.1, 65.5)
- moved C201 172.8 mm to (131.2, 92.8), turned to 180 degrees
- moved R403 171.9 mm to (160.0, 68.1), turned to 180 degrees
- moved R201 165.3 mm to (134.7, 92.8), turned to 270 degrees
- moved C202 164.4 mm to (135.3, 89.0), turned to 180 degrees
- moved R501 163.3 mm to (134.2, 59.1)
- moved R401 162.3 mm to (160.0, 69.7)
- moved D201 160.5 mm to (135.0, 87.0), turned to 180 degrees
- moved L201 160.0 mm to (131.2, 87.0)
- moved R402 158.0 mm to (160.0, 71.5)
- moved U201 155.5 mm to (131.2, 90.0), turned to 180 degrees
- moved C401 147.4 mm to (176.9, 82.2)
- moved C402 147.2 mm to (179.2, 72.3), turned to 180 degrees
- moved J102 147.1 mm to (181.9, 58.2), turned to 180 degrees
- moved R405 145.9 mm to (185.4, 78.7), turned to 270 degrees
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Connections:
- C201 pad 1: +2V8 -> GND
- C202 pad 2: +2V8 -> GND
- C301 pad 2: +2V8 -> GND
- C302 pad 2: +2V8 -> GND
- C303 pad 2: +2V8 -> GND
- C304 pad 2: +2V8 -> GND
- C305 pad 1: +2V8 -> GND
- C308 pad 2: +2V8 -> GND
- C309 pad 2: +2V8 -> GND
- C310 pad 2: +2V8 -> GND
- C311 pad 2: +2V8 -> GND
- C312 pad 2: +2V8 -> GND
- C401 pad 1: +2V8 -> GND
- C402 pad 2: +2V8 -> GND
- C501 pad 1: GNDPWR -> /Power/Vin
- C501 pad 2: /Power/Vin -> GND
- C502 pad 2: GNDPWR -> GND
- C504 pad 1: +2V8 -> GND
- C505 pad 2: +2V8 -> GND
- C506 pad 2: +2V8 -> GND
- C507 pad 2: Net-(C507-Pad2) -> GND
- C510 pad 1: /Coulomb Counter/Vbatt_source -> Net-(C507-Pad1)
- C510 pad 2: +2V8 -> GND
- D102 pad 1: +2V8 -> GND
- F101 pad 1: /Power/Vext -> Net-(F101-Pad1)
- F102 pad 2: Net-(F102-Pad2) -> Net-(C102-Pad1)
- FB301 pad 2: +2V8 -> GND
- J101 pad 2: GNDPWR -> GND
- J103 pad 2: +2V8 -> GND
- J104 pad 2: +2V8 -> GND
- J201 pad 10: +2V8 -> GND
- J201 pad 11: +2V8 -> GND
- J201 pad 12: +2V8 -> GND
- J201 pad 13: +2V8 -> GND
- J201 pad 14: +2V8 -> GND
- J201 pad 15: +2V8 -> GND
- J201 pad 16: +2V8 -> GND
- J201 pad 17: +2V8 -> GND
- J201 pad 18: +2V8 -> GND
- J201 pad 19: +2V8 -> GND
- J201 pad 2: +2V8 -> GND
- J201 pad 20: +2V8 -> GND
- J201 pad 21: +2V8 -> GND
- J201 pad 22: +2V8 -> GND
- J201 pad 23: +2V8 -> GND
- J201 pad 24: +2V8 -> GND
- J201 pad 25: +2V8 -> GND
- J201 pad 26: +2V8 -> GND
- J201 pad 27: +2V8 -> GND
- J201 pad 28: +2V8 -> GND
- J201 pad 29: /(Opt) TFT Display/SDI -> /(Opt) TFT Display/SDO
- J201 pad 33: +2V8 -> /(Opt) TFT Display/D~CX
- J201 pad 38: +2V8 -> GND
- J201 pad 39: +2V8 -> GND
- J201 pad 7: +2V8 -> GND
- J201 pad 8: +2V8 -> GND
- J201 pad 9: +2V8 -> GND
- J301 pad 3: +2V8 -> GND
- J301 pad 5: +2V8 -> GND
- J301 pad 9: +2V8 -> GND
- J302 pad 1: +2V8 -> GND
- J302 pad 10: +2V8 -> GND
- J302 pad 2: +2V8 -> /Microcontroller/PB8
- J302 pad 3: Net-(J302-Pad3) -> +2V8
- J302 pad 4: /Microcontroller/CC_~AL~CC -> +2V8
- J302 pad 5: /Microcontroller/SPI1_SCK -> /Microcontroller/TFT_~CS
- J302 pad 6: /Microcontroller/SPI1_MOSI -> /(Opt) TFT Display/D~CX
- J302 pad 7: /Microcontroller/SPI1_MISO -> /(Opt) TFT Display/SCL
- J302 pad 8: /Microcontroller/SPI1_NSS -> /(Opt) TFT Display/SDI
- J302 pad 9: +2V8 -> /(Opt) TFT Display/SDO
- J303 pad 1: +2V8 -> GND
- J303 pad 10: +2V8 -> GND
- J303 pad 2: +2V8 -> /Microcontroller/SPI1_NSS
- J303 pad 3: /Microcontroller/PA8 -> /Microcontroller/SPI1_SCK
- J303 pad 4: /Microcontroller/PB8 -> /Microcontroller/Vadj
- J303 pad 5: /(Opt) TFT Display/SCL -> /Microcontroller/SPI1_MISO
- J303 pad 6: /(Opt) TFT Display/SDI -> /Microcontroller/SPI1_MOSI
- J303 pad 7: /(Opt) TFT Display/SDI -> /Microcontroller/PB9
- J303 pad 8: /Microcontroller/TFT_~CS -> /Microcontroller/CC_SDA
- J303 pad 9: +2V8 -> /Microcontroller/CC_SCL
- L501 pad 1: Net-(C507-Pad2) -> Net-(C503-Pad2)
- L501 pad 2: /Coulomb Counter/Vbatt_source -> Net-(C507-Pad1)
- Q101 pad 1: Net-(Q101-Pad1) -> GND
- Q101 pad 2: +5V -> /Power/Vin
- Q101 pad 3: /Power/Vin -> Net-(F101-Pad1)
- R101 pad 1: /Power/Vext -> Net-(C101-Pad1)
- R101 pad 2: Net-(Q101-Pad1) -> GND
- R102 pad 1: Net-(Q101-Pad1) -> /Power/Vin
- R102 pad 2: +2V8 -> Net-(J101-Pad3)
- R201 pad 2: +2V8 -> GND
- R406 pad 2: /Coulomb Counter/Vbatt_source -> Net-(Q403-Pad5)
- R501 pad 2: /Microcontroller/Pgood -> /Power/En
- R502 pad 1: +2V8 -> Net-(R502-Pad1)
- R502 pad 2: /Power/En -> GND
- R503 pad 1: /Power/Vext -> Net-(R502-Pad1)
- R503 pad 2: +2V8 -> /Microcontroller/Vadj
- R504 pad 1: Net-(C507-Pad2) -> Net-(R502-Pad1)
- R504 pad 2: Net-(R504-Pad2) -> Net-(C507-Pad1)
- SW301 pad 2: +2V8 -> GND
- SW302 pad 2: +2V8 -> GND
- SW303 pad 2: +2V8 -> GND
- SW304 pad 2: +2V8 -> GND
- U201 pad 2: +2V8 -> GND
- U301 pad 4: +2V8 -> GND
- U302 pad 10: /Microcontroller/CC_~AL~CC -> Net-(R315-Pad2)
- U302 pad 11: /Microcontroller/Pgood -> /Microcontroller/CC_~5mA
- U302 pad 19: Net-(D301-Pad1) -> /Microcontroller/CC_~500mA
- U302 pad 21: +2V8 -> /(Opt) TFT Display/D~CX
- U302 pad 23: +2V8 -> GND
- U302 pad 27: /(Opt) TFT Display/SDI -> /(Opt) TFT Display/SDO
- U302 pad 29: /Microcontroller/PA8 -> /Microcontroller/CC_~AL~CC
- U302 pad 32: /Microcontroller/USB_DM -> /USB_N
- U302 pad 33: /Microcontroller/USB_DP -> /USB_P
- U302 pad 35: +2V8 -> GND
- U302 pad 38: Net-(U302-Pad38) -> /Microcontroller/CC_~50mA
- U302 pad 46: Net-(U302-Pad46) -> /Microcontroller/PB9
- U302 pad 47: +2V8 -> GND
- U302 pad 49: +2V8 -> GND
- U401 pad 2: +2V8 -> GND
- U501 pad 1: Net-(C503-Pad2) -> GND
- U501 pad 3: Net-(R504-Pad2) -> /Power/Vin
- U501 pad 4: Net-(Q503-Pad1) -> Net-(R502-Pad1)
- U501 pad 5: GNDPWR -> /Power/En
- U501 pad 6: /Power/Vin -> Net-(C503-Pad1)
- U502 pad 1: +2V8 -> GND
Routing:
- net GND: track 0.00 -> 248.3 mm, vias 0 -> 33
- net +2V8: track 0.00 -> 186.4 mm, vias 0 -> 32
- net /Power/Vin: track 0.00 -> 129.6 mm, vias 0 -> 16
- net /Microcontroller/Vadj: track 0.00 -> 99.1 mm, vias 0 -> 4
- net /Microcontroller/CC_SDA: track 0.00 -> 97.3 mm, vias 0 -> 6
- net /Microcontroller/CC_SCL: track 0.00 -> 95.5 mm, vias 0 -> 6
- net /Microcontroller/CC_~5mA: track 0.00 -> 93.7 mm, vias 0 -> 2
- net /Power/En: track 0.00 -> 91.0 mm, vias 0 -> 2
- net /Coulomb Counter/Vbatt_source: track 0.00 -> 82.3 mm, vias 0 -> 3
- net /Microcontroller/CC_~500mA: track 0.00 -> 72.3 mm, vias 0 -> 2
- net /(Opt) TFT Display/D~CX: track 0.00 -> 71.3 mm, vias 0 -> 2
- net /(Opt) TFT Display/SDO: track 0.00 -> 66.3 mm, vias 0 -> 2
- net /(Opt) TFT Display/SCL: track 0.00 -> 63.8 mm, vias 0 -> 2
- net /(Opt) TFT Display/SDI: track 0.00 -> 62.7 mm, vias 0 -> 2
- net /Microcontroller/CC_~50mA: track 0.00 -> 60.7 mm, vias 0 -> 2
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- added copper zone on B.Cu, net +2V8
- added copper zone on F.Cu, net +2V8
- added copper zone on B.Cu, net /Coulomb Counter/Vbatt_out
- added copper zone on F.Cu, net /Coulomb Counter/Vbatt_out
- added copper zone on B.Cu, net /Coulomb Counter/Vbatt_source
- added copper zone on B.Cu, net /Power/Vin
- added copper zone on F.Cu, net /Power/Vin
- added copper zone on B.Cu, net GND
- added copper zone on F.Cu, net GND
- added copper zone on F.Cu, net Net-(C101-Pad1)
- added copper zone on F.Cu, net Net-(F101-Pad2)
Other:
- board size 160 x 106.7 mm -> 78.1 x 62.2 mm
- net class Default: clearance 0.2 -> 0.1; via_dia 0.8 -> 0.4; via_drill 0.4 -> 0.2
- rule trace_clearance: 0.2 -> 0.1
- rule trace_min: 0.2 -> 0.1
- rule via_min_drill: 0.3 -> 0.2
- board text added: "+"
- board text added: "-"
- board text added: "2V8"
- board text added: "GND"
- board text added: "MISO"
- board text added: "MOSI"
- board text added: "NanoBat v0.1.0"
- board text added: "PB8"
- board text added: "PB9"
- board text added: "PWR"
- board text added: "SCK"
- board text added: "SCL"
- board text added: "SDA"
- board text added: "STAT"
- board text added: "Serial Number"
- board text added: "TD~CX"
- board text added: "TSCL"
- board text added: "TSDI"
- board text added: "TSDO"
- board text added: "T~CS"
- board text added: "Vadj"
- board text added: "Vertigo Designs"
- board text added: "~CS"
